File: eagle/DC25_HHV_RE-A.sch (EAGLE design)
At the start: 21 parts, among them U1 PIC12F1571

Commit message: Added BOM
Parts:
- R1, R2, R3, R4: value (none) -> 10k
- S1: value 0 -> B3F-10XX
- S2: value 1 -> B3F-10XX
- S3: value 2 -> B3F-10XX
- S4: value 3 -> B3F-10XX
Changed lines of the file:
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@@
 <part name="C1" library="rcl" deviceset="C-EU" device="050-024X044" value=".1uF"/>
 <part name="VSS2" library="supply1" deviceset="VSS" device=""/>
-<part name="S1" library="switch-omron" deviceset="10-XX" device="" value="0"/>
-<part name="S2" library="switch-omron" deviceset="10-XX" device="" value="1"/>
-<part name="S3" library="switch-omron" deviceset="10-XX" device="" value="2"/>
-<part name="S4" library="switch-omron" deviceset="10-XX" device="" value="3"/>
-<part name="R2" library="rcl" deviceset="R-US_" device="0207/10"/>
-<part name="R3" library="rcl" deviceset="R-US_" device="0207/10"/>
-<part name="R4" library="rcl" deviceset="R-US_" device="0207/10"/>
-<part name="R1" library="rcl" deviceset="R-US_" device="0207/10"/>
+<part name="S1" library="switch-omron" deviceset="10-XX" device="" value="B3F-10XX"/>
+<part name="S2" library="switch-omron" deviceset="10-XX" device="" value="B3F-10XX"/>
+<part name="S3" library="switch-omron" deviceset="10-XX" device="" value="B3F-10XX"/>
+<part name="S4" library="switch-omron" deviceset="10-XX" device="" value="B3F-10XX"/>
+<part name="R2" library="rcl" deviceset="R-US_" device="0207/10" value="10k"/>
+<part name="R3" library="rcl" deviceset="R-US_" device="0207/10" value="10k"/>
+<part name="R4" library="rcl" deviceset="R-US_" device="0207/10" value="10k"/>
+<part name="R1" library="rcl" deviceset="R-US_" device="0207/10" value="10k"/>
 <part name="VSS3" library="supply1" deviceset="VSS" device=""/>
 <part name="VSS4" library="supply1" deviceset="VSS" device=""/>
